Commit message: include hand in urdf

File: polymetis/polymetis/data/franka_panda/panda_arm.urdf (robot description, URDF)
Before this commit: robot panda, 9 links, 8 joints
Links:
- added link panda_hand; collision mesh filename=meshes/collision/hand.stl; visual mesh filename=meshes/visual/hand.dae
- added link panda_leftfinger; collision mesh filename=meshes/collision/finger.stl; visual mesh filename=meshes/visual/finger.dae
- added link panda_rightfinger; collision mesh filename=meshes/collision/finger.stl; visual mesh filename=meshes/visual/finger.dae
Joints:
- added joint panda_finger_joint1: type prismatic, parent panda_hand, child panda_leftfinger, origin xyz=0 0 0.0584 rpy=0 0 0, axis 0 1 0, limit lower=-0.001 upper=0.04 effort=20 velocity=0.3
- added joint panda_finger_joint2: type prismatic, parent panda_hand, child panda_rightfinger, origin xyz=0 0 0.0584 rpy=0 0 0, axis 0 -1 0, limit lower=-0.001 upper=0.04 effort=20 velocity=0.3
- added joint panda_hand_joint: type fixed, parent panda_link8, child panda_hand, origin xyz=0 0 0 rpy=0 0 -0.785398163397

Commit message: remove panda hand joint

File: polymetis/polymetis/data/franka_panda/panda_arm.urdf (robot description, URDF)
Before this commit: robot panda, 12 links, 11 joints
Links:
- removed link panda_hand
- removed link panda_leftfinger
- removed link panda_rightfinger
Joints:
- removed joint panda_finger_joint1
- removed joint panda_finger_joint2
- removed joint panda_hand_joint
- removed joint panda_joint8

Commit message: Recover arm joint

File: polymetis/polymetis/data/franka_panda/panda_arm.urdf (robot description, URDF)
Before this commit: robot panda, 9 links, 7 joints
Joints:
- added joint panda_joint8: type fixed, parent panda_link7, child panda_link8, origin xyz=0 0 0.107 rpy=0 0 0, axis 0 0 0
